Commit message: tbot3_webots: Fix urdf and add visual files locally

File: tbot3_webots/description/urdf/turtlebot3_waffle.urdf (robot description, URDF)
Before this commit: robot turtlebot3_waffle, 13 links, 12 joints
Links:
- removed link camera_depth_frame
- removed link camera_depth_optical_frame
- removed link camera_link
- removed link camera_rgb_frame
- removed link camera_rgb_optical_frame
- link base_link: geometry collision box size=0.266 0.266 0.094; visual mesh filename=package://tbot3_webots/description/meshes/collision/waffle_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 scale=0.001 0.001 0.001
- link base_scan: geometry collision cylinder length=0.0315 radius=0.055; visual mesh filename=package://tbot3_webots/description/meshes/collision/lds.stl scale=0.001 0.001 0.001
- link wheel_left_link: geometry collision cylinder length=0.018 radius=0.033; visual mesh filename=package://tbot3_webots/description/meshes/collision/left_ti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 scale=0.001 0.001 0.001
- link wheel_right_link: geometry collision cylinder length=0.018 radius=0.033; visual mesh filename=package://tbot3_webots/description/meshes/collision/right_t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 scale=0.001 0.001 0.001
Joints:
- removed joint camera_depth_joint
- removed joint camera_depth_optical_joint
- removed joint camera_joint
- removed joint camera_rgb_joint
- removed joint camera_rgb_optical_joint

Commit message: urdf: Use dae files for visual elements

File: tbot3_webots/description/urdf/turtlebot3_waffle.urdf (robot description, URDF)
Before this commit: robot turtlebot3_waffle, 7 links, 6 joints
Links:
- link base_link: geometry collision box size=0.266 0.266 0.094; visual mesh filename=package://tbot3_webots/description/meshes/visual/waffle_bas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 scale=0.001 0.001 0.001
- link wheel_left_link: geometry collision cylinder length=0.018 radius=0.033; visual mesh filename=package://tbot3_webots/description/meshes/visual/left_tire.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 scale=0.001 0.001 0.001
- link wheel_right_link: geometry collision cylinder length=0.018 radius=0.033; visual mesh filename=package://tbot3_webots/description/meshes/visual/right_tire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 scale=0.001 0.001 0.001

Commit message: Fix proto workflow solution

File: tbot3_webots/description/urdf/turtlebot3_waffle.urdf (robot description, URDF)
Before this commit: robot turtlebot3_waffle, 7 links, 6 joints
Links:
- removed link base_scan
- removed link caster_back_left_link
- removed link caster_back_right_link
- removed link imu_link
Joints:
- removed joint caster_back_left_joint
- removed joint caster_back_right_joint
- removed joint imu_joint
- removed joint scan_joint
