Commit message: webots: Add base_scan frame in URDF

File: tbot3_webots/description/urdf/turtlebot3_waffle_clean.urdf (robot description, URDF)
Before this commit: robot turtlebot3_waffle, 3 links, 2 joints
Links:
- added link base_scan
Joints:
- added joint base_scan_joint: type fixed, parent base_link, child base_scan, origin xyz=0 0 0.1 rpy=0 0 0

Commit message: clearn urdf: Update base_scan position

File: tbot3_webots/description/urdf/turtlebot3_waffle_clean.urdf (robot description, URDF)
Before this commit: robot turtlebot3_waffle, 4 links, 3 joints
Joints:
- joint base_scan_joint: origin xyz=0 0 0.1 rpy=0 0 0 -> xyz=0 0 0.2 rpy=0 0 0
